Commit message: added URDF

File: amr_robots_description/urdf/pioneer3dx.urdf (robot description, URDF)
Before this commit: robot pioneer3dx, 11 links, 10 joints
Links:
- added link robot_base
Joints:
- added joint robot_base_to_base_link: type fixed, parent robot_base, child base_link, origin xyz=0 0 0 rpy=0 0 0
