Commit message: 20251012

File: amr_robots_description/urdf/pioneer3dx_gazebo.urdf.xacro (robot description, xacro)
@@ -26,5 +26,5 @@
 			<origin xyz="-0.045 0 0.148" rpy="0 0 0"/>
 			<geometry name="pioneer_geom">
-				<mesh filename="package://amr_robots_description/meshes/p3dx_meshes/chassis.stl"/>
+				<mesh filename="package://meshes/p3dx_meshes/chassis.stl"/>
 			</geometry>
 			<material name="ChassisRed">
@@ -50,5 +50,5 @@
 			<origin xyz="0 0 0" rpy="0 0 0"/>
 			<geometry name="pioneer_geom">
-				<mesh filename="package://amr_robots_description/meshes/p3dx_meshes/top.stl"/>
+				<mesh filename="package://meshes/p3dx_meshes/top.stl"/>
 			</geometry>
 			<material name="TopBlack">
@@ -77,5 +77,5 @@
 			<origin xyz="0 0 0" rpy="0 0 0"/>
 			<geometry name="pioneer_geom">
-				<mesh filename="package://amr_robots_description/meshes/p3dx_meshes/front_sonar.stl"/>
+				<mesh filename="package://meshes/p3dx_meshes/front_sonar.stl"/>
 			</geometry>
 			<material name="SonarYellow">
@@ -107,5 +107,5 @@
 			<origin xyz="0 0 0" rpy="0 0 0"/>
 			<geometry name="pioneer_geom">
-				<mesh filename="package://amr_robots_description/meshes/p3dx_meshes/back_sonar.stl"/>
+				<mesh filename="package://meshes/p3dx_meshes/back_sonar.stl"/>
 			</geometry>
 			<material name="SonarYellow">
@@ -133,5 +133,5 @@
 		<origin xyz="0 0 0" rpy="0 0 0"/>
 		<geometry name="pioneer_geom">
-			<mesh filename="package://amr_robots_description/meshes/p3dx_meshes/caster_swivel.stl"/>
+			<mesh filename="package://meshes/p3dx_meshes/caster_swivel.stl"/>
 		</geometry>
 		<material name="caster_swivel">
@@ -154,5 +154,5 @@
 		<origin xyz="0 0 0" rpy="0 0 0"/>
 		<geometry name="pioneer_geom">
-			<mesh filename="package://amr_robots_description/meshes/p3dx_meshes/caster_hubcap.stl"/>
+			<mesh filename="package://meshes/p3dx_meshes/caster_hubcap.stl"/>
 		</geometry>
 		<material name="caster_swivel">
@@ -189,5 +189,5 @@
 		<origin xyz="0 0 0" rpy="0 0 0"/>
 		<geometry name="pioneer_geom">
-			<mesh filename="package://amr_robots_description/meshes/p3dx_meshes/caster_wheel.stl"/>
+			<mesh filename="package://meshes/p3dx_meshes/caster_wheel.stl"/>
 		</geometry>
 		<material name="WheelBlack">
@@ -198,5 +198,5 @@
 		<origin xyz="0 0 0" rpy="${-3.1415927/2.0} 0 0"/>
 		<geometry>
-			<!--<mesh filename="package://amr_robots_description/meshes/p3dx_meshes/caster_wheel.stl"/>-->
+			<!--<mesh filename="package://meshes/p3dx_meshes/caster_wheel.stl"/>-->
 			<cylinder radius="0.0375" length="0.01"/>
 		</geometry>
@@ -215,5 +215,5 @@
 			<origin xyz="0 0 0" rpy="0 0 0"/>
 			<geometry>
-				<mesh filename="package://amr_robots_description/meshes/p3dx_meshes/left_hubcap.stl"/>
+				<mesh filename="package://meshes/p3dx_meshes/left_hubcap.stl"/>
 			</geometry>
 			<material name="HubcapYellow">
@@ -224,5 +224,5 @@
 			<origin xyz="0 0 0" rpy="${-3.1415927/2.0} 0 0"/>
 			<geometry>
-				<!--<mesh filename="package://amr_robots_description/meshes/p3dx_meshes/caster_wheel.stl"/>-->
+				<!--<mesh filename="package://meshes/p3dx_meshes/caster_wheel.stl"/>-->
 				<cylinder radius="0.09" length="0.01"/>
 			</geometry>
@@ -239,5 +239,5 @@
 			<origin xyz="0 0 0" rpy="0 0 0"/>
 			<geometry>
-				<mesh filename="package://amr_robots_description/meshes/p3dx_meshes/left_wheel.stl"/>
+				<mesh filename="package://meshes/p3dx_meshes/left_wheel.stl"/>
 			</geometry>
 			<material name="WheelBlack">
@@ -258,5 +258,5 @@
 			<origin xyz="0 0 0" rpy="0 0 0"/>
 			<geometry>
-				<mesh filename="package://amr_robots_description/meshes/p3dx_meshes/right_hubcap.stl"/>
+				<mesh filename="package://meshes/p3dx_meshes/right_hubcap.stl"/>
 			</geometry>
 			<material name="HubcapYellow">
@@ -267,5 +267,5 @@
 		<origin xyz="0 0 0" rpy="${-3.1415927/2.0} 0 0"/>
 		<geometry>
-			<!--<mesh filename="package://amr_robots_description/meshes/p3dx_meshes/caster_wheel.stl"/>-->
+			<!--<mesh filename="package://meshes/p3dx_meshes/caster_wheel.stl"/>-->
 			<cylinder radius="0.09" length="0.01"/>
 		</geometry>
@@ -285,5 +285,5 @@
 			<origin xyz="0 0 0" rpy="0 0 0"/>
 			<geometry>
-				<mesh filename="package://amr_robots_description/meshes/p3dx_meshes/right_wheel.stl"/>
+				<mesh filename="package://meshes/p3dx_meshes/right_wheel.stl"/>
 			</geometry>
 			<material name="WheelBlack">

Commit message: 20251013

File: amr_robots_description/urdf/pioneer3dx_gazebo.urdf.xacro (robot description, xacro)
@@ -246,8 +246,10 @@
 		</visual>
 	</link>
-	<joint name="left_wheel_joint" type="fixed"> <!-- type="continuous" -->
+	<joint name="left_wheel_joint" type="continuous" >
 		<origin xyz="0 0 0" rpy="0 0 0"/>
 		<parent link="left_hub"/>
 		<child link="left_wheel"/>
+		<axis   xyz="0 1 0"/> <!-- pas as aan als nodig -->
+  		<limit effort="5.0" velocity="20.0"/>
 	</joint>
 	<gazebo reference="left_wheel_joint">
@@ -292,8 +294,10 @@
 		</visual>
 	</link>
-	<joint name="right_wheel_joint" type="fixed"> <!-- type="continuous" -->
+	<joint name="right_wheel_joint" type="continuous" >
 		<origin xyz="0 0 0" rpy="0 0 0"/>
 		<parent link="right_hub"/>
 		<child link="right_wheel"/>
+		<axis   xyz="0 1 0"/> <!-- pas as aan als nodig -->
+  		<limit effort="5.0" velocity="20.0"/>
 	</joint>
 	<gazebo reference="right_wheel_joint">
@@ -304,37 +308,19 @@
   	<top_plate  parent="base_link"/>
   	</create>
-	<!-- Changed by Gerard-->
-	<gazebo>
-	<!-- Differential drive plugin -->
-	<plugin name="differential_drive_controller" filename="libgazebo_ros_diff_drive.so">
-		<alwaysOn>true</alwaysOn>
-		<updateRate>100</updateRate>
-		<leftJoint>left_wheel_joint</leftJoint>
-		<rightJoint>right_wheel_joint</rightJoint>
-		<wheelSeparation>0.158</wheelSeparation>
-		<wheelDiameter>0.12</wheelDiameter>
-		<torque>5</torque>
-		<!-- Optional: specify joint velocity/position interfaces -->
-		<!-- <interface>velocity</interface> -->
-		<commandTopic>cmd_vel</commandTopic>
-		<robotBaseFrame>base_link</robotBaseFrame>
-		<odometryTopic>odom</odometryTopic>
-		<odometryFrame>odom</odometryFrame>
-	</plugin>
-	<!-- Ground truth pose (P3D) plugin -->
-	<plugin name="ground_truth_pose" filename="libgazebo_ros_p3d.so">
-		<alwaysOn>true</alwaysOn>
-		<updateRate>50</updateRate>
-		<bodyName>base_link</bodyName>
-		<topicName>ground_truth</topicName>
-		<frameName>odom</frameName>
-	</plugin>
-	<!-- Optional: controller manager (ROS 2 example) -->
-	<!--
-	<plugin name="ros2_controller_manager" filename="libgazebo_ros2_control.so">
-		<robotNamespace>/</robotNamespace>
-		<controlPeriod>0.01</controlPeriod>
-	</plugin>
-	-->
-	</gazebo>
+	<!-- ============================= -->
+	<!-- Ignition Gazebo Diff Drive Plugin -->
+	<!-- ============================= -->
+  <gazebo>
+    <plugin name="diff_drive_plugin" filename="libignition-gazebo-diff-drive-system.so">
+      <left_joint>left_wheel_joint</left_joint>
+      <right_joint>right_wheel_joint</right_joint>
+      <wheel_separation>0.3</wheel_separation>
+      <wheel_radius>0.09</wheel_radius>
+      <topic>/model/pioneer3dx/cmd_vel</topic>
+      <enable_odom>true</enable_odom>
+      <odom_frame>odom</odom_frame>
+      <base_frame>base_link</base_frame>
+      <publish_rate>50</publish_rate>
+    </plugin>
+  </gazebo>
 </robot>
