Commit message: 20251012

File: amr_robots_description/urdf/pioneer3dx.urdf.xacro (robot description, xacro)
@@ -7,4 +7,5 @@
   <!--<include filename="$(find amr_robots_description)/urdf/materials.xacro"/>-->
   <xacro:include filename="$(find amr_robots_description)/urdf/pioneer3dx_wheel.xacro"/>
+  <xacro:include filename="$(find amr_robots_description)/urdf/materials.xacro"/>
 <!-- Chassis -->
 	<link name="base_link">
@@ -111,7 +112,9 @@
 	<joint name="base_caster_swivel_joint" type="continuous">
 		<origin xyz="-0.185 0 0.055" rpy="0 0 0"/>
+		<!--
 		<anchor xyz="0 0 0"/>
     	<limit effort="100" velocity="100" k_velocity="0" />
     	<joint_properties damping="0.0" friction="0.0" />
+		-->
 		<parent link="base_link"/>
 		<child link="caster_swivel"/>
@@ -124,18 +127,18 @@
 				 iyy="0.01" iyz="0" izz="0.01"/>
   	 	</inertial>
-	<visual>
-		<origin xyz="0 0 0" rpy="0 0 0"/>
-		<geometry name="pioneer_geom">
-			<mesh filename="package://amr_robots_description/meshes/p3dx_meshes/caster_swivel.stl"/>
-		</geometry>
-		<material name="caster_swivel">
-			<color rgba="0.5 0.5 0.5 1"/>
-		</material>
-	</visual>
+		<visual>
+			<origin xyz="0 0 0" rpy="0 0 0"/>
+			<geometry name="pioneer_geom">
+				<mesh filename="package://amr_robots_description/meshes/p3dx_meshes/caster_swivel.stl"/>
+			</geometry>
+			<material name="caster_swivel">
+				<color rgba="0.5 0.5 0.5 1"/>
+			</material>
+		</visual>
 	</link>
 	<gazebo reference="caster_swivel">
 		<material value="Gazebo/Grey"/>
 	</gazebo>
-<!-- Center Wheel + Hubcap -->
+	<!-- Center Wheel + Hubcap -->
 	<link name="caster_hubcap">
 		<inertial>
@@ -150,5 +153,5 @@
 			<mesh filename="package://amr_robots_description/meshes/p3dx_meshes/caster_hubcap.stl"/>
 		</geometry>
-		<material name="caster_swivel">
+		<material name="caster_hubcap">
 			<color rgba="0.5 0.5 0.5 1"/>
 		</material>
@@ -166,9 +169,14 @@
 	<joint name="caster_swivel_hubcap_joint" type="continuous">
 		<origin xyz="-0.026 0 -0.016" rpy="0 0 0"/>
+		<!--
 		<axis xyz="0 1 0"/>
 		<anchor xyz="0 0 0"/>
-    <limit effort="100" velocity="100" k_velocity="0" />
-    <joint_properties damping="0.0" friction="0.0" />
-	  <parent link="caster_swivel"/>
+		<limit effort="100" velocity="100" k_velocity="0" />
+		<joint_properties damping="0.0" friction="0.0" />
+		-->
+		<parent link="base_link"/>
+		<!--
+		<parent link="caster_swivel"/>
+		-->
 		<child link="caster_wheel"/>
 	</joint>
@@ -190,5 +198,8 @@
 	</visual>
 	<collision>
+		<!-->
 		<origin xyz="0 0 0" rpy="${-3.1415927/2.0} 0 0"/>
+		-->
+		<origin xyz="0 0 0" rpy="-1.57079635 0 0"/>
 		<geometry>
 			<!--<mesh filename="package://amr_robots_description/meshes/p3dx_meshes/caster_wheel.stl"/>-->
@@ -216,5 +227,8 @@
 		</visual>
 		<collision>
+			<!--
 			<origin xyz="0 0 0" rpy="${-3.1415927/2.0} 0 0"/>
+			-->
+			<origin xyz="0 0 0" rpy="-1.57079635 0 0"/>
 			<geometry>
 				<!--<mesh filename="package://amr_robots_description/meshes/p3dx_meshes/caster_wheel.stl"/>-->
@@ -259,5 +273,8 @@
 		</visual>
 		<collision>
+		<!--
 		<origin xyz="0 0 0" rpy="${-3.1415927/2.0} 0 0"/>
+		-->
+		<origin xyz="0 0 0" rpy="-1.57079635 0 0"/>
 		<geometry>
 			<!--<mesh filename="package://amr_robots_description/meshes/p3dx_meshes/caster_wheel.stl"/>-->

File: amr_robots_description/urdf/pioneer3dx_body.xacro (robot description, xacro)
@@ -145,5 +145,8 @@
 	</visual>
 	<collision>
+		<!--
 		<origin xyz="0 0 0" rpy="${-3.1415927/2.0} 0 0"/>
+		-->
+		<origin xyz="0 0 0" rpy="-1.57079635 0 0"/>
 		<geometry>
 			<!--<mesh filename="package://amr_robots_description/meshes/p3dx_meshes/center_wheel.stl"/>-->
@@ -171,5 +174,8 @@
 		</visual>
 		<collision>
+			<!--
 			<origin xyz="0 0 0" rpy="${-3.1415927/2.0} 0 0"/>
+			-->
+			<origin xyz="0 0 0" rpy="-1.57079635 0 0"/>
 			<geometry>
 				<!--<mesh filename="package://amr_robots_description/meshes/p3dx_meshes/center_wheel.stl"/>-->
@@ -214,5 +220,8 @@
 		</visual>
 		<collision>
+		<!--
 		<origin xyz="0 0 0" rpy="${-3.1415927/2.0} 0 0"/>
+		-->
+		<origin xyz="0 0 0" rpy="-1.57079635 0 0"/>
 		<geometry>
 			<!--<mesh filename="package://amr_robots_description/meshes/p3dx_meshes/center_wheel.stl"/>-->

File: amr_robots_description/urdf/pioneer3dx_wheel.xacro (robot description, xacro)
@@ -28,5 +28,8 @@
     </visual>
     <collision>
+      <!--
       <origin xyz="0 0 0" rpy="${-3.1415927/2} 0 0"/>
+      -->
+      <origin xyz="0 0 0" rpy="-1.57079635 0 0"/>
       <geometry>
         <!--<mesh filename="package://amr_robots_description/meshes/p3dx_meshes/${suffix}_wheel.stl"/>-->

Commit message: 20251014

File: amr_robots_description/urdf/pioneer3dx.urdf.xacro (robot description, xacro)
@@ -246,5 +246,5 @@
 		</visual>
 	</link>
-	<joint name="left_wheel_joint" type="fixed"> <!-- type="continuous" -->
+	<joint name="left_wheel_joint" type="continuous" >
 		<origin xyz="0 0 0" rpy="0 0 0"/>
 		<parent link="left_hub"/>
@@ -292,5 +292,5 @@
 		</visual>
 	</link>
-	<joint name="right_wheel_joint" type="fixed"> <!-- type="continuous" -->
+	<joint name="right_wheel_joint" type="continuous">
 		<origin xyz="0 0 0" rpy="0 0 0"/>
 		<parent link="right_hub"/>
@@ -304,37 +304,21 @@
   	<top_plate  parent="base_link"/>
   	</create>
-	<!-- Changed by Gerard-->
-	<gazebo>
-	<!-- Differential drive plugin -->
-	<plugin name="differential_drive_controller" filename="libgazebo_ros_diff_drive.so">
-		<alwaysOn>true</alwaysOn>
-		<updateRate>100</updateRate>
-		<leftJoint>left_wheel_joint</leftJoint>
-		<rightJoint>right_wheel_joint</rightJoint>
-		<wheelSeparation>0.158</wheelSeparation>
-		<wheelDiameter>0.12</wheelDiameter>
-		<torque>5</torque>
-		<!-- Optional: specify joint velocity/position interfaces -->
-		<!-- <interface>velocity</interface> -->
-		<commandTopic>cmd_vel</commandTopic>
-		<robotBaseFrame>base_link</robotBaseFrame>
-		<odometryTopic>odom</odometryTopic>
-		<odometryFrame>odom</odometryFrame>
-	</plugin>
-	<!-- Ground truth pose (P3D) plugin -->
-	<plugin name="ground_truth_pose" filename="libgazebo_ros_p3d.so">
-		<alwaysOn>true</alwaysOn>
-		<updateRate>50</updateRate>
-		<bodyName>base_link</bodyName>
-		<topicName>ground_truth</topicName>
-		<frameName>odom</frameName>
-	</plugin>
-	<!-- Optional: controller manager (ROS 2 example) -->
-	<!--
-	<plugin name="ros2_controller_manager" filename="libgazebo_ros2_control.so">
-		<robotNamespace>/</robotNamespace>
-		<controlPeriod>0.01</controlPeriod>
-	</plugin>
-	-->
-	</gazebo>
+	<!-- ============================= -->
+	<!-- Ignition Gazebo Diff Drive Plugin -->
+	<!-- ============================= -->
+  <gazebo>
+    <plugin
+		filename="gz-sim-diff-drive-system"
+		name="gz::sim::systems::DiffDrive">
+		<left_joint>left_wheel_joint</left_joint>
+		<right_joint>right_wheel_joint</right_joint>
+		<wheel_separation>0.3</wheel_separation>
+		<wheel_radius>0.09</wheel_radius>
+		<topic>/model/pioneer3dx/cmd_vel</topic>
+		<enable_odom>true</enable_odom>
+		<odom_frame>odom</odom_frame>
+		<base_frame>base_link</base_frame>
+		<publish_rate>50</publish_rate>
+    </plugin>
+  </gazebo>
 </robot>

Commit message: 20251014

File: amr_robots_description/urdf/pioneer3dx.urdf.xacro (robot description, xacro)
@@ -174,7 +174,7 @@
 		<axis xyz="0 1 0"/>
 		<anchor xyz="0 0 0"/>
-    <limit effort="100" velocity="100" k_velocity="0" />
-    <joint_properties damping="0.0" friction="0.0" />
-	  <parent link="caster_swivel"/>
+		<limit effort="100" velocity="100" k_velocity="0" />
+		<joint_properties damping="0.0" friction="0.0" />
+	  	<parent link="caster_swivel"/>
 		<child link="caster_wheel"/>
 	</joint>
@@ -211,15 +211,17 @@
 		<child link="caster_hubcap"/>
 	</joint>
-	<link name="left_hub">
-		<visual>
-			<origin xyz="0 0 0" rpy="0 0 0"/>
-			<geometry>
-				<mesh filename="package://amr_robots_description/meshes/p3dx_meshes/left_hubcap.stl"/>
-			</geometry>
-			<material name="HubcapYellow">
-				<color rgba="1.0 0.811 0.151 1.0"/>
-			</material>
-		</visual>
-		<collision>
+	<!-- Wheels -->
+	<xacro:macro name="wheel" params="prefix y_offset">
+		<link name="${prefix}_hub">
+			<visual>
+				<origin xyz="0 0 0" rpy="0 0 0"/>
+				<geometry>
+					<mesh filename="package://amr_robots_description/meshes/p3dx_meshes/${prefix}_hubcap.stl"/>
+				</geometry>
+				<material name="HubcapYellow">
+					<color rgba="1.0 0.811 0.151 1.0"/>
+				</material>
+			</visual>
+			<collision>
 			<origin xyz="0 0 0" rpy="${-3.1415927/2.0} 0 0"/>
 			<geometry>
@@ -228,76 +230,52 @@
 			</geometry>
 		</collision>
-	</link>
-	<joint name="left_hub_joint" type="fixed">
-		<origin xyz="0 0.15 0.08" rpy="0 0 0"/>
-		<parent link="base_link"/>
-		<child link="left_hub"/>
-		<axis xyz="0 1 0"/>
-	</joint>
-	<link name="left_wheel">
-		<visual>
-			<origin xyz="0 0 0" rpy="0 0 0"/>
-			<geometry>
-				<mesh filename="package://amr_robots_description/meshes/p3dx_meshes/left_wheel.stl"/>
-			</geometry>
-			<material name="WheelBlack">
-				<color rgba="0.117 0.117 0.117 1"/>
-			</material>
-		</visual>
-	</link>
-	<joint name="left_wheel_joint" type="continuous" >
-		<origin xyz="0 0 0" rpy="0 0 0"/>
-		<parent link="left_hub"/>
-		<child link="left_wheel"/>
-	</joint>
-	<gazebo reference="left_wheel_joint">
-		<material value="Gazebo/Black"/>
-	</gazebo>
-	<link name="right_hub">
-		<visual>
-			<origin xyz="0 0 0" rpy="0 0 0"/>
-			<geometry>
-				<mesh filename="package://amr_robots_description/meshes/p3dx_meshes/right_hubcap.stl"/>
-			</geometry>
-			<material name="HubcapYellow">
-				<color rgba="1.0 0.811 0.151 1.0"/>
-			</material>
-		</visual>
-		<collision>
-		<origin xyz="0 0 0" rpy="${-3.1415927/2.0} 0 0"/>
-		<geometry>
-			<!--<mesh filename="package://amr_robots_description/meshes/p3dx_meshes/caster_wheel.stl"/>-->
-			<cylinder radius="0.09" length="0.01"/>
-		</geometry>
-	</collision>
-	</link>
-	<gazebo reference="right_hub">
-		<material value="Gazebo/Yellow"/>
-	</gazebo>
-	<joint name="right_hub_joint" type="fixed">
-		<origin xyz="0 -0.15 0.08" rpy="0 0 0"/>
-		<parent link="base_link"/>
-		<child link="right_hub"/>
-		<axis xyz="0 1 0"/>
-	</joint>
-	<link name="right_wheel">
-		<visual>
-			<origin xyz="0 0 0" rpy="0 0 0"/>
-			<geometry>
-				<mesh filename="package://amr_robots_description/meshes/p3dx_meshes/right_wheel.stl"/>
-			</geometry>
-			<material name="WheelBlack">
-				<color rgba="0.117 0.117 0.117 1"/>
-			</material>
-		</visual>
-	</link>
-	<joint name="right_wheel_joint" type="continuous">
-		<origin xyz="0 0 0" rpy="0 0 0"/>
-		<parent link="right_hub"/>
-		<child link="right_wheel"/>
-	</joint>
-	<gazebo reference="right_wheel_joint">
-		<material value="Gazebo/Black"/>
-	</gazebo>
+		</link>
+		<gazebo reference="${prefix}_hub">
+			<material value="Gazebo/Yellow"/>
+		</gazebo>
+		<joint name="${prefix}_hub_joint" type="fixed">
+			<origin xyz="0 ${y_offset} 0.08" rpy="0 0 0"/>
+			<parent link="base_link"/>
+			<child link="${prefix}_hub"/>
+			<axis xyz="0 1 0"/>
+		</joint>
+		<link name="${prefix}_wheel">
+			<visual>
+				<origin xyz="0 0 0" rpy="0 0 0"/>
+				<geometry>
+					<mesh filename="package://amr_robots_description/meshes/p3dx_meshes/${prefix}_wheel.stl"/>
+					<cylinder>
+						<radius>0.12</radius>
+						<length>0.04</length>
+					</cylinder>
+				</geometry>
+				<material name="WheelBlack">
+					<color rgba="0.117 0.117 0.117 1"/>
+				</material>
+			</visual>
+		</link>
+		<gazebo reference="${prefix}_wheel">
+			<material value="Gazebo/Black"/>
+		</gazebo>
+		<joint name="${prefix}_wheel_joint" type="revolute">
+			<origin xyz="0 0 0" rpy="0 0 0"/>
+			<axis>
+			<xyz>0 1 0</xyz>
+			<limit>
+				<lower>-inf</lower>
+				<upper>inf</upper>
+			</limit>
+			</axis>
+			<limit effort="100" velocity="100" k_velocity="0" />
+			<joint_properties damping="0.0" friction="0.0" />
+			<parent link="${prefix}_hub"/>
+			<child link="${prefix}_wheel"/>
+		</joint>
+		<gazebo reference="${prefix}_wheel_joint">
+			<material value="Gazebo/Black"/>
+		</gazebo>
+	</xacro:macro>
+	<xacro:wheel prefix="left" y_offset="0.15" />
+	<xacro:wheel prefix="right" y_offset="-0.15" />
 	<create>
 	<back_sonar parent="base_link"/>
@@ -307,28 +285,31 @@
 	<!-- Ignition Gazebo Diff Drive Plugin -->
 	<!-- ============================= -->
-  <gazebo>
-    <plugin
-		filename="gz-sim-diff-drive-system"
-		name="gz::sim::systems::DiffDrive">
-		<left_joint>left_wheel_joint</left_joint>
-		<right_joint>right_wheel_joint</right_joint>
-		<wheel_separation>0.158</wheel_separation>
-      	<wheel_radius>0.12</wheel_radius>
-		<!--
-		<wheel_separation>0.3</wheel_separation>
-		<wheel_radius>0.09</wheel_radius>
-		-->
-		<topic>/model/pioneer3dx/cmd_vel</topic>
-		<!--
-		<enable_odom>true</enable_odom>
-		<odom_frame>odom</odom_frame>
-		-->
-		<base_frame>base_link</base_frame>
-		<publish_rate>50</publish_rate>
-    </plugin>
-	<plugin
-		name="gz::sim::systems::JointStatePublisher"
-		filename="libgz-sim-joint-state-publisher-system.so">
-	</plugin>
-  </gazebo>
+	<gazebo>
+		<plugin
+			filename="gz-sim-diff-drive-system"
+			name="gz::sim::systems::DiffDrive">
+			<left_joint>pioneer3dx::left_wheel_joint</left_joint>
+			<right_joint>pioneer3dx::right_wheel_joint</right_joint>
+			<wheel_separation>0.158</wheel_separation>
+			<wheel_radius>0.12</wheel_radius>
+			<!--
+			<wheel_separation>0.3</wheel_separation>
+			<wheel_radius>0.09</wheel_radius>
+			-->
+			<!--
+			<topic>/model/pioneer3dx/cmd_vel</topic>
+			-->
+			<!--
+			<enable_odom>true</enable_odom>
+			<odom_frame>odom</odom_frame>
+			-->
+			<base_frame>base_link</base_frame>
+			<publish_rate>50</publish_rate>
+			<publish_joint_states>true</publish_joint_states>
+		</plugin>
+		<plugin
+			name="gz::sim::systems::JointStatePublisher"
+			filename="libgz-sim-joint-state-publisher-system.so">
+		</plugin>
+	</gazebo>
 </robot>
