Commit message: 20251016

File: amr_gazebo/models/robots/pioneer3dx.sdf.xacro (robot description, xacro)
@@ -23,6 +23,7 @@
     <pose>0 0 0 0 0 0</pose>
     -->
-    <!-- Base Link / Chassis -->
-    <link name="base_link">
+    <link name="base_link"/>
+    <!-- Chassis -->
+    <link name="chassis">
       <pose>0 0 0 0 0 0</pose>
       <inertial>
@@ -39,12 +40,19 @@
       <visual name="chassis_visual">
         <geometry>
+          <!--
+          <box>
+            <size>0.01 0.01 0.01</size>
+          </box>
+          -->
           <mesh>
             <uri>package://amr_robots_description/meshes/p3dx_meshes/chassis.stl</uri>
           </mesh>
         </geometry>
+        <!--
         <material>
           <ambient>0.851 0 0 1</ambient>
           <diffuse>0.851 0 0 1</diffuse>
         </material>
+        -->
       </visual>
       <collision name="chassis_collision">
@@ -56,4 +64,9 @@
       </collision>
     </link>
+    <joint name="chassis_joint" type="fixed">
+      <parent>base_link</parent>
+      <child>chassis</child>
+      <pose>0 0 0 0 0 0</pose>
+    </joint>
     <!-- Top Plate -->
     <link name="top_plate">
@@ -178,5 +191,5 @@
     <!-- Wheels & Hub -->
     <xacro:macro name="wheel" params="prefix y_offset">
-      <!-- Right Hub & Wheel -->
+      <!-- Wheel Hub -->
       <link name="${prefix}_hub">
         <pose>0 ${y_offset} 0.08 0 0 0</pose>
@@ -192,41 +205,38 @@
         <parent>base_link</parent>
         <child>${prefix}_hub</child>
-        <pose>0 -0.15 0.08 0 0 0</pose>
       </joint>
+      <!-- Wheel -->
       <link name="${prefix}_wheel">
-        <pose>0 0 0 0 0 0</pose>
-          <visual name="${prefix}_wheel_visual">
-            <geometry>
-              <!--
-              <mesh>
-                <uri>model://amr_robots_description/meshes/p3dx_meshes/${prefix}_wheel.stl</uri>
-              </mesh>
-                -->
-              <cylinder>
-                <radius>${wheel_radius}</radius>
-                <length>${wheel_width}</length>
-              </cylinder>
-            </geometry>
-            <material>
-              <ambient>0.3 0.3 0.3 1.0</ambient>
-              <diffuse>0.7 0.7 0.7 1.0</diffuse>
-            </material>
-          </visual>
-      <xacro:cylinder_inertia m="0.5" r="${wheel_radius}" h="${wheel_width}"/>
+        <pose>0 ${y_offset} 0.08 0 0 0</pose> <!-- dit snap ik niet  -->
+        <visual name="${prefix}_wheel_visual">
+          <geometry>
+            <mesh>
+              <uri>package://amr_robots_description/meshes/p3dx_meshes/${prefix}_wheel.stl</uri>
+            </mesh>
+          </geometry>
+          <material>
+            <ambient>0.3 0.3 0.3 1.0</ambient>
+            <diffuse>0.7 0.7 0.7 1.0</diffuse>
+          </material>
+        </visual>
+        <!-- Wheel inertia -->
+        <xacro:cylinder_inertia m="0.5" r="${wheel_radius}" h="${wheel_width}"/>
       </link>
+      <!-- Revolute joint for wheel rotation -->
       <joint name="${prefix}_wheel_joint" type="revolute">
         <parent>${prefix}_hub</parent>
         <child>${prefix}_wheel</child>
-        <!--
-        <axis><xyz>0 1 0</xyz></axis>
-        -->
+        <!-- Move wheel along x so it lines up properly with hub -->
+        <pose>0 0 0 0 0 0</pose>
+        <!-- Rotation axis along Y -->
         <axis>
-            <xyz>0 1 0</xyz>
-            <limit>
-              <lower>-1e16</lower>
-              <upper>1e16</upper>
-            </limit>
+          <xyz>0 1 0</xyz>
+          <limit>
+            <lower>-1e16</lower>
+            <upper>1e16</upper>
+            <effort>10</effort>
+            <velocity>10</velocity>
+          </limit>
         </axis>
-        <pose>0 0 0 -1.57079635 0 0</pose> <!-- ???? -->
       </joint>
     </xacro:macro>
@@ -234,4 +244,5 @@
     <xacro:wheel prefix="right" y_offset="-0.15" />
     <!-- DiffDrive Plugin -->
+    <!--
     <plugin
       filename="gz-sim-diff-drive-system"
@@ -245,9 +256,12 @@
       <publish_joint_states>true</publish_joint_states>
     </plugin>
+    -->
     <!-- JointState Publisher -->
+    <!--
     <plugin
       name="gz::sim::systems::JointStatePublisher"
       filename="libgz-sim-joint-state-publisher-system.so">
     </plugin>
+    -->
   </model>
 </sdf>

File: amr_robots_description/urdf/pioneer3dx.urdf.xacro (robot description, xacro)
@@ -226,5 +226,5 @@
 			<origin xyz="0 0 0" rpy="${-3.1415927/2.0} 0 0"/>
 			<geometry>
-				<!--<mesh filename="package://amr_robots_description/meshes/p3dx_meshes/caster_wheel.stl"/>-->
+				<!--<mesh filename="package://amr_robots_description/meshes/p3dx_meshes/${prefix}_wheel.stl"/>-->
 				<cylinder radius="0.09" length="0.01"/>
 			</geometry>
@@ -245,8 +245,10 @@
 				<geometry>
 					<mesh filename="package://amr_robots_description/meshes/p3dx_meshes/${prefix}_wheel.stl"/>
+					<!--
 					<cylinder>
 						<radius>0.12</radius>
 						<length>0.04</length>
 					</cylinder>
+					-->
 				</geometry>
 				<material name="WheelBlack">
@@ -258,5 +260,5 @@
 			<material value="Gazebo/Black"/>
 		</gazebo>
-		<joint name="${prefix}_wheel_joint" type="revolute">
+		<joint name="${prefix}_wheel_joint" type="fixed"> <!--type="revolute"-->
 			<origin xyz="0 0 0" rpy="0 0 0"/>
 			<axis>
@@ -279,6 +281,6 @@
 	<xacro:wheel prefix="right" y_offset="-0.15" />
 	<create>
-	<back_sonar parent="base_link"/>
-  	<top_plate  parent="base_link"/>
+		<back_sonar parent="base_link"/>
+		<top_plate  parent="base_link"/>
   	</create>
 	<!-- ============================= -->

Commit message: 20251016

File: amr_gazebo/models/robots/pioneer3dx.sdf.xacro (robot description, xacro)
@@ -23,7 +23,5 @@
     <pose>0 0 0 0 0 0</pose>
     -->
-    <link name="base_link"/>
-    <!-- Chassis -->
-    <link name="chassis">
+    <link name="base_link">
       <pose>0 0 0 0 0 0</pose>
       <inertial>
@@ -40,19 +38,12 @@
       <visual name="chassis_visual">
         <geometry>
-          <!--
-          <box>
-            <size>0.01 0.01 0.01</size>
-          </box>
-          -->
-          <mesh>
-            <uri>package://amr_robots_description/meshes/p3dx_meshes/chassis.stl</uri>
-          </mesh>
-        </geometry>
-        <!--
+          <mesh>
+            <uri>package://amr_robots_description/meshes/p3dx_meshes/chassisx.stl</uri>
+          </mesh>
+        </geometry>
         <material>
           <ambient>0.851 0 0 1</ambient>
           <diffuse>0.851 0 0 1</diffuse>
         </material>
-        -->
       </visual>
       <collision name="chassis_collision">
@@ -64,4 +55,5 @@
       </collision>
     </link>
+<!--
     <joint name="chassis_joint" type="fixed">
       <parent>base_link</parent>
@@ -69,4 +61,5 @@
       <pose>0 0 0 0 0 0</pose>
     </joint>
+-->
     <!-- Top Plate -->
     <link name="top_plate">
